Commit message: Configurations en simulationsfiles ready

File: ros2_ws/src/ur10_pbvs_sim/urdf/ur10_camera.urdf.xacro (robot description, xacro)
@@ -42,9 +42,9 @@
    <xacro:arg name="use_fake_hardware" default="false" />
    <xacro:arg name="fake_sensor_commands" default="false" />
-   <xacro:arg name="sim_gazebo" default="false" />
+   <xacro:arg name="sim_gazebo" default="true" />
    <xacro:arg name="sim_ignition" default="false" />
-   <xacro:arg name="simulation_controllers" default="" />
+   <xacro:arg name="simulation_controllers" default="$(find ur10_pbvs_sim)/config/ur10_controllers.yaml" />
    <!-- initial position for simulations (Fake Hardware, Gazebo, Ignition) -->
-   <xacro:arg name="initial_positions_file" default="$(find ur_description)/config/initial_positions.yaml"/>
+   <xacro:arg name="initial_positions_file" default="$(find ur10_pbvs_sim)/config/initial_positions.yaml"/>
    <!-- convert to property to use substitution in function -->
    <xacro:property name="initial_positions_file" default="$(arg initial_positions_file)"/>
@@ -115,5 +115,5 @@
      trajectory_port="$(arg trajectory_port)"
      >
-     <origin xyz="0 0 0" rpy="0 0 0" />          <!-- position robot in the world -->
+     <origin xyz="0 0 0.8" rpy="0 0 0" />          <!-- position robot in the world -->
    </xacro:ur_robot>
    <xacro:if value="$(arg sim_gazebo)">

Commit message: Camera added to URDF

File: ros2_ws/src/ur10_pbvs_sim/urdf/ur10_camera.urdf.xacro (robot description, xacro)
@@ -5,4 +5,5 @@
    <!-- import main macro -->
    <xacro:include filename="$(find ur10_pbvs_sim)/urdf/ur10_macro.xacro"/>
+   <!--<xacro:include filename="$(find ur10_pbvs_sim)/urdf/wrist_camera.xacro"/> -->
    <!-- possible 'ur_type' values: ur3, ur5, ur10, ur3e, ur5e, ur7e, ur10e, ur12e, ur16e, ur8long, ur15, ur18, ur20, ur30 -->
    <!-- the default value should raise an error in case this was called without defining the type -->
@@ -138,3 +139,71 @@
     </gazebo>
   </xacro:if>
+ <!-- CAMERA ATTACHMENT -->
+ <joint name="wrist_camera_link_joint" type="fixed">
+  <origin xyz="0 0 0.05" rpy="0 0 0"/>
+  <parent link="wrist_3_link"/>
+  <child link="wrist_camera_link"/>
+</joint>
+<link name="wrist_camera_link">
+     <visual>
+    <origin xyz="0 0 0" rpy="0 0 0"/>
+    <geometry>
+      <box size="0.02 0.02 0.02"/>
+    </geometry>
+    <material name="camera_material">
+      <color rgba="0.1 0.1 0.1 1"/>
+    </material>
+  </visual>
+  <collision>
+    <origin xyz="0 0 0" rpy="0 0 0"/>
+    <geometry>
+      <box size="0.02 0.02 0.02"/>
+    </geometry>
+  </collision>
+  <inertial>
+    <mass value="0.01"/>
+    <origin xyz="0 0 0"/>
+    <inertia
+      ixx="1e-6" ixy="0" ixz="0"
+      iyy="1e-6" iyz="0"
+      izz="1e-6"/>
+  </inertial>
+</link>
+<gazebo reference="wrist_camera_link">
+  <sensor type="camera" name="wrist_camera_sensor">
+    <update_rate>30</update_rate>
+    <visualize>true</visualize>
+    <camera>
+      <horizontal_fov>1.396</horizontal_fov>
+      <image>
+        <width>640</width>
+        <height>480</height>
+        <format>R8G8B8</format>
+      </image>
+      <clip>
+        <near>0.02</near>
+        <far>5.0</far>
+      </clip>
+      <noise>
+        <type>gaussian</type>
+        <mean>0.0</mean>
+        <stddev>0.007</stddev>
+      </noise>
+    </camera>
+    <plugin name="camera_plugin" filename="libgazebo_ros_camera.so">
+      <ros>
+        <namespace>/wrist_camera</namespace>
+        <remapping>image_raw:=image</remapping>
+      </ros>
+      <frame_name>wrist_camera_link</frame_name>
+    </plugin>
+  </sensor>
+</gazebo>
+<!--
+  <xacro:wrist_camera
+      parent_link="tool0"
+      xyz="0 0 0.05"
+      rpy="0 0 0"
+      sim_gazebo="$(arg sim_gazebo)"/>
+-->
 </robot>
